File: shutdownPCB/AIR_OUTPUT.kicad_sch (KiCad schematic)
At the start: 20 parts, among them K1 APAN3103, K2 APAN3103, K3 APAN3103, K4 APAN3103, K5 APAN3103, Q5 BC816-25HVL, Q6 BC816-25HVL, Q7 BC816-25HVL, Q8 BC816-25HVL, Q9 BC816-25HVL

Commit message: Updated 12 Sep
Parts:
- added AMS_REL1, BSPD_REL1, DRV_OUT_REL1, IMD_REL1, PDOC_REL1: TestPoint, TestPoint:TestPoint_Pad_D2.0mm, symbol Connector:TestPoint
- added D10, D11, D2, D3, D9: 1N4148W RHG, UniSA_Motorsport_Diode:SOD-123F-2, symbol UniSA_Motorsport_Diode:1N4148W_RHG
Connections:
- net 3.3V: now also D2.1 (K)
- net 3.3V_0: now also D3.1 (K)
- net 3.3V_1: now also D9.1 (K)
- net 3.3V_2: now also D10.1 (K)
- net 3.3V_PDOC: now also D11.1 (K)
- net SAFTEY_OUT: now also PDOC_REL1.1
- net at K5.1, Q9.3: now also D10.2 (A)
- net at K3.1, Q7.3: now also D2.2 (A)
- net at K2.3, K3.4: now also DRV_OUT_REL1.1
- net at K2.1, Q6.3: now also D3.2 (A)
- net at K4.1, Q8.3: now also D11.2 (A)
- net at K1.1, Q5.3: now also D9.2 (A)
- net at K1.3, K2.4: now also AMS_REL1.1
- net at K1.4, K5.3: now also IMD_REL1.1
- net at K4.3, K5.4: now also BSPD_REL1.1
Other:
- note added: "PDOC"
