File: shutdownPCB/NonDriverResetableInputs.kicad_sch (KiCad schematic)
At the start: 88 parts, among them Q1 SI2318DS-T1-BE3, Q2 SI2318DS-T1-BE3, Q3 SI2318DS-T1-BE3, Q4 SI2318DS-T1-BE3, U10 MC74AC02DR2G, U11 MC74AC02DR2G, U12 74AUP1G32GW,125, U13 74AUP1G32GW,125, U14 74AHC1GU04GW,125, U16 MC74AC02DR2G, U17 74AHC1GU04GW,125, U18 MC74AC02DR2G, U19 CD4071BM96, U20 74LVC1G08GW,125, U21 74LVC1G08GW,125, U23 74AHC1GU04GW,125, U24 74AHC1GU04GW,125, U9 TC7S04FU,LF

Commit message: Updated 12 Sep
Parts:
- added U22, U26, U27, U28, U29, U30, U31: SN74LVC1G126, UniSA_Motorsport_SO:SC70-5, symbol UniSA_Motorsport_Logic:SN74LVC1G126_
- 1K1: renamed from R43; Resistance 150R -> 1000k
- R21, R22, R23, R82: Resistance 150R -> 220R
- R42, R44: Resistance 150R -> 1K
- renumbered LED1 to LED3, LED1 to LED4, LED1 to LED5, LED1 to LED6, LED1 to LED7, LED1 to LED8, LED1 to LED9
Connections:
- net 3.3V_0: now also U26.1, U26.5
- net 3.3V_1: now also U22.1, U22.5
- net 3.3V_2: now also U27.1, U27.5
- net 3.3V_PDOC: now also U28.1, U28.5, U29.1, U29.5, U30.1, U30.5, U31.1, U31.5
- net AMS_LED: now also U26.4; no longer R24.2, U10.2, U10.3, U9.4
- net BSPD_LED: now also U27.4; no longer R26.2, U13.4, U16.2, U16.3
- net GND: now also U22.3, U26.3, U27.3, U28.3, U29.3, U30.3, U31.3
- net HV_IMD_LED: now also U22.4; no longer R25.2, U11.2, U11.3, U12.4
- net HV_PDOC_LED: now also U31.4; no longer R45.2, U19.3
- net MA_PDOC_LED: now also U30.4; no longer R46.2, U19.4
- net PDOC_LED: now also U29.4; no longer R51.2, U18.2, U18.3, U21.4
- net SA_PDOC_LED: now also U28.4; no longer R47.2, U19.10
- new net: R51.2, U18.2, U18.3, U21.4, U29.2
- new net: R46.2, U19.4, U30.2
- new net: R26.2, U13.4, U16.2, U16.3, U27.2
- new net: R24.2, U10.2, U10.3, U26.2, U9.4
- new net: R47.2, U19.10, U28.2
- new net: R45.2, U19.3, U31.2
- new net: R25.2, U11.2, U11.3, U12.4, U22.2
Other:
- moved on the sheet: 1K1, LED3, LED4, LED5, LED6, LED7, LED8, LED9, R21, R22, R23, R42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
