File: shutdownPCB/connector.kicad_sch (KiCad schematic)
At the start: 6 parts, among them J2 HLE-108-02-L-DV-BE-K-TR, J3 HLE-108-02-L-DV-BE-K-TR, J4 HLE-108-02-L-DV-BE-K-TR, J5 43045-2215, J5 HLE-108-02-L-DV-BE-K-TR

Commit message: Updated 12 Sep
Connections:
- net GLV_MASTER_SWITCH_OUT: no longer J2.14 (Pin_14), J2.15 (Pin_15), J2.16 (Pin_16)
- net DRIVER_OUTPUT renamed DRIVER_OUTPUT_LED
- net SHOULDER_OUT renamed SHOULDER_OUT_LED
- no-connect marks 34 -> 37
