File: shutdownPCB/feather.kicad_sch (KiCad schematic)
At the start: 57 parts, among them U15 CD4051BM96G3, U25 CD4051BM96G3

Commit message: Updated 12 Sep
Parts:
- added U34: SN74LVC1G126, UniSA_Motorsport_SO:SC70-5, symbol UniSA_Motorsport_Logic:SN74LVC1G126_
- R75: Resistance 150R -> 220R
- renumbered LED1 to LED10, LED1 to LED11, LED1 to LED12, LED1 to LED13, LED1 to LED14, LED1 to LED15, LED1 to LED16, LED1 to LED17, LED1 to LED18, LED1 to LED19, LED1 to LED20
Connections:
- net 3.3V: now also U34.1, U34.5
- net FEATHER_OUT: now also U34.4; no longer A1.5 (A0)
- net GND: now also U34.3
- new net: A1.5 (A0), U34.2
