File: shutdownPCB/logic.kicad_sch (KiCad schematic)
At the start: 26 parts, among them U21 74LVC1G08GW,125, U4 74AHC1GU04GW,125, U5 MC14013BDR2G, U7 74AHC1GU04GW,125

Commit message: Updated 12 Sep
Parts:
- added U32, U33: SN74LVC1G126, UniSA_Motorsport_SO:SC70-5, symbol UniSA_Motorsport_Logic:SN74LVC1G126_
- R4, R7: Resistance 150R -> 220R
- renumbered C19 to C45, U21 to U1, U21 to U2, U21 to U3, U21 to U6, U21 to U8
Connections:
- net 3.3V: now also U32.1, U32.5, U33.1, U33.5
- net DRIVER_OUTPUT: now also U33.2; no longer R7.1
- net GND: now also U32.3, U33.3
- net SHOULDER_OUT: no longer names the net of PRES_1.1, U5.1 (Q), U6.2
- net SHOULDER_OUT: now also U32.2; no longer R4.1
- new net DRIVER_OUTPUT_LED: R7.1, U33.4
- new net SHOULDER_OUT_LED: R4.1, U32.4
Other:
- moved on the sheet: C45, LED1, LED2, R4, R7, U5C
