File: shutdownPCB/powerRegulation.kicad_sch (KiCad schematic)
At the start: 55 parts

Commit message: Updated 12 Sep
Parts:
- renumbered PRES_1 to BREAK_PRESSED1, R39 to R10, R39 to R11, R39 to R16, R39 to R17, R39 to R18, R39 to R36, R39 to R37, R39 to R38, R39 to R8, R39 to R9
Connections:
- net 3.3V: now also R8.1
- net 3.3V_0: now also R37.1
- net 3.3V_1: now also R10.1
- net 3.3V_2: now also R16.1
- net 3.3V_PDOC: now also R18.1
- net at C24.2, L2.1, PS2.6 (SW): no longer R10.1
- net at C30.2, L3.1, PS3.6 (SW): no longer R16.1
- net at C7.2, L1.1, PS1.6 (SW): no longer R8.1
- net at C42.2, L5.1, PS5.6 (SW): no longer R37.1
- net at C36.2, L4.1, PS4.6 (SW): no longer R18.1
- net at R37.2, R38.1: no longer PS5.1 (VFB)
Other:
- moved on the sheet: BREAK_PRESSED1, C25, C26, C31, C32, C37, C38, C43, C44, C8, C9, R10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
