File: shutdownPCB/shutdownPCB.kicad_pcb (KiCad board)
At the start: 2 copper layers, 152 x 141.4 mm, 257 parts, among them J1 HLE-108-02-L-DV-BE-K-TR, J2 HLE-108-02-L-DV-BE-K-TR, J3 HLE-108-02-L-DV-BE-K-TR, J4 HLE-108-02-L-DV-BE-K-TR, J5 43045-2215, K1 APAN3103, K2 APAN3103, K3 APAN3103, K4 APAN3103, K5 APAN3103, Q1 SI2318DS-T1-BE3, Q2 SI2318DS-T1-BE3, Q3 SI2318DS-T1-BE3, Q4 SI2318DS-T1-BE3, Q5 BC816-25HVL, Q6 BC816-25HVL, Q7 BC816-25HVL, Q8 BC816-25HVL, Q9 BC816-25HVL, U1 74LVC1G08GW,125, U10 MC74AC02DR2G, U11 MC74AC02DR2G, U12 74AUP1G32GW,125, U13 74AUP1G32GW,125, U14 74AHC1GU04GW,125, U15 CD4051BM96G3, U16 MC74AC02DR2G, U17 74AHC1GU04GW,125, U18 MC74AC02DR2G, U19 CD4071BM96, U2 74LVC1G08GW,125, U20 74LVC1G08GW,125, U21 74LVC1G08GW,125, U23 74AHC1GU04GW,125, U24 74AHC1GU04GW,125, U25 CD4051BM96G3, U3 74LVC1G08GW,125, U4 74AHC1GU04GW,125, U5 MC14013BDR2G, U6 74LVC1G08GW,125, U7 74AHC1GU04GW,125, U8 74LVC1G08GW,125, U9 TC7S04FU,LF

Commit message: Updated 12 Sep
Parts:
- added AMS_REL1: TestPoint, TestPoint:TestPoint_Pad_D2.0mm, F.Cu at (215.0, 163.6)
- added BSPD_REL1: TestPoint, TestPoint:TestPoint_Pad_D2.0mm, F.Cu at (215.0, 178.4)
- added D10: 1N4148W RHG, UniSA_Motorsport_Diode:SOD-123F-2, F.Cu at (188.4, 177.4)
- added D11: 1N4148W RHG, UniSA_Motorsport_Diode:SOD-123F-2, F.Cu at (188.0, 186.3)
- added D2: 1N4148W RHG, UniSA_Motorsport_Diode:SOD-123F-2, F.Cu at (188.1, 153.8)
- added D3: 1N4148W RHG, UniSA_Motorsport_Diode:SOD-123F-2, F.Cu at (188.2, 161.6)
- added D9: 1N4148W RHG, UniSA_Motorsport_Diode:SOD-123F-2, F.Cu at (188.0, 169.4)
- added DRV_OUT_REL1: TestPoint, TestPoint:TestPoint_Pad_D2.0mm, F.Cu at (215.0, 155.5)
- added IMD_REL1: TestPoint, TestPoint:TestPoint_Pad_D2.0mm, F.Cu at (215.1, 170.7)
- added PDOC_REL1: TestPoint, TestPoint:TestPoint_Pad_D2.0mm, F.Cu at (214.6, 187.4)
- added U22: SN74LVC1G126, UniSA_Motorsport_SO:SC70-5, F.Cu at (113.5, 187.2)
- added U26: SN74LVC1G126, UniSA_Motorsport_SO:SC70-5, F.Cu at (104.3, 172.2)
- added U27: SN74LVC1G126, UniSA_Motorsport_SO:SC70-5, F.Cu at (109.6, 203.2)
- added U28: SN74LVC1G126, UniSA_Motorsport_SO:SC70-5, F.Cu at (168.6, 189.1)
- added U29: SN74LVC1G126, UniSA_Motorsport_SO:SC70-5, F.Cu at (135.5, 188.2)
- added U30: SN74LVC1G126, UniSA_Motorsport_SO:SC70-5, F.Cu at (162.8, 165.8)
- added U31: SN74LVC1G126, UniSA_Motorsport_SO:SC70-5, F.Cu at (170.5, 178.6)
- added U32: SN74LVC1G126, UniSA_Motorsport_SO:SC70-5, F.Cu at (162.5, 210.1)
- added U33: SN74LVC1G126, UniSA_Motorsport_SO:SC70-5, F.Cu at (162.5, 206.2)
- added U34: SN74LVC1G126, UniSA_Motorsport_SO:SC70-5, F.Cu at (199.7, 89.6)
- moved R62 4.00 mm to (179.4, 168.9)
- moved Q5 4.00 mm to (183.2, 170.2)
- moved R59 4.00 mm to (179.4, 171.1)
- moved R60 3.85 mm to (179.3, 163.0)
- moved R63 3.85 mm to (179.3, 160.8)
- moved Q6 3.85 mm to (183.1, 162.1)
- moved Q9 3.82 mm to (183.4, 178.0)
- moved R66 3.82 mm to (179.6, 178.9)
- moved R77 3.82 mm to (179.6, 176.7)
- moved R65 3.66 mm to (179.7, 186.9)
- moved Q8 3.66 mm to (183.5, 186.0)
- moved R76 3.66 mm to (179.7, 184.7)
- moved Q7 3.34 mm to (183.4, 153.6)
- moved R64 3.34 mm to (179.6, 152.3)
- moved R61 3.34 mm to (179.6, 154.5)
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- renumbered R43 to 1K1, 24V1 to 24V, 3.3V_PDOC1 to 3.3V_PDOC, AMS_LED1 to AMS_LED, BSPD_LED1 to BSPD_LED, DRIVER_OUTPUT1 to DRIVER_OUTPUT, FIX_AMS1 to FIX_AMS, FIX_BSPD1 to FIX_BSPD, FIX_IMD1 to FIX_IMD, FIX_PDOC1 to FIX_PDOC, FIX_PDOC_HV1 to FIX_PDOC_HV, FIX_PDOC_MAS1 to FIX_PDOC_MAS, FIX_PDOC_SLAVE1 to FIX_PDOC_SLAVE, GND1 to GND, IMD_LED1 to IMD_LED, NON_RESETS1 to NON_RESETS, NON_RESETS_OUT1 to NON_RESETS_OUT, PDOC_LED1 to PDOC_LED, SHOULDER_RESET1 to SHOULDER_RESET
Connections:
- net /connector/DASH_E-STOP_OUT renamed /connector/DASH_ESTOP_OUT
- A1 pad 5: /connector/FEATHER_OUT -> Net-(A1-A0)
- J1 pad 14: /connector/GLV_MASTER_SWITCH_OUT -> unconnected-(J1-Pin_14-Pad14)
- J1 pad 15: /connector/GLV_MASTER_SWITCH_OUT -> unconnected-(J1-Pin_15-Pad15)
- J1 pad 16: /connector/GLV_MASTER_SWITCH_OUT -> unconnected-(J1-Pin_16-Pad16)
- J5 pad 1: /AIR_OUTPUT/DRIVER_OUTPUT -> /connector/DRIVER_OUTPUT_LED
- J5 pad 2: /connector/SHOULDER_OUT -> /connector/SHOULDER_OUT_LED
- NON_RESETS_OUT pad 1: /connector/SHOULDER_OUT -> Net-(U5A-Q)
- R10 pad 1: Net-(PS2-SW) -> /3.3V_1
- R16 pad 1: Net-(PS3-SW) -> /3.3V_2
- R18 pad 1: Net-(PS4-SW) -> /3.3V_PDOC
- R24 pad 2: /NonDriverResetableInputs/AMS_LED -> Net-(R24-Pad2)
- R25 pad 2: /NonDriverResetableInputs/HV_IMD_LED -> Net-(R25-Pad2)
- R26 pad 2: /NonDriverResetableInputs/BSPD_LED -> Net-(R26-Pad2)
- R37 pad 1: Net-(PS5-SW) -> /3.3V_0
- R4 pad 1: /connector/SHOULDER_OUT -> /connector/SHOULDER_OUT_LED
- R45 pad 2: /NonDriverResetableInputs/HV_PDOC_LED -> Net-(R45-Pad2)
- R46 pad 2: /NonDriverResetableInputs/MA_PDOC_LED -> Net-(R46-Pad2)
- R47 pad 2: /NonDriverResetableInputs/SA_PDOC_LED -> Net-(R47-Pad2)
- R51 pad 2: /NonDriverResetableInputs/PDOC_LED -> Net-(R51-Pad2)
- R7 pad 1: /AIR_OUTPUT/DRIVER_OUTPUT -> /connector/DRIVER_OUTPUT_LED
- R8 pad 1: Net-(PS1-SW) -> /3.3V
- U10 pad 2: /NonDriverResetableInputs/AMS_LED -> Net-(R24-Pad2)
- U10 pad 3: /NonDriverResetableInputs/AMS_LED -> Net-(R24-Pad2)
- U11 pad 2: /NonDriverResetableInputs/HV_IMD_LED -> Net-(R25-Pad2)
- U11 pad 3: /NonDriverResetableInputs/HV_IMD_LED -> Net-(R25-Pad2)
- U12 pad 4: /NonDriverResetableInputs/HV_IMD_LED -> Net-(R25-Pad2)
- U13 pad 4: /NonDriverResetableInputs/BSPD_LED -> Net-(R26-Pad2)
- U16 pad 2: /NonDriverResetableInputs/BSPD_LED -> Net-(R26-Pad2)
- U16 pad 3: /NonDriverResetableInputs/BSPD_LED -> Net-(R26-Pad2)
- U18 pad 2: /NonDriverResetableInputs/PDOC_LED -> Net-(R51-Pad2)
- U18 pad 3: /NonDriverResetableInputs/PDOC_LED -> Net-(R51-Pad2)
- U19 pad 10: /NonDriverResetableInputs/SA_PDOC_LED -> Net-(R47-Pad2)
- U19 pad 3: /NonDriverResetableInputs/HV_PDOC_LED -> Net-(R45-Pad2)
- U19 pad 4: /NonDriverResetableInputs/MA_PDOC_LED -> Net-(R46-Pad2)
- U21 pad 4: /NonDriverResetableInputs/PDOC_LED -> Net-(R51-Pad2)
- U5 pad 1: /connector/SHOULDER_OUT -> Net-(U5A-Q)
- U6 pad 2: /connector/SHOULDER_OUT -> Net-(U5A-Q)
- U9 pad 4: /NonDriverResetableInputs/AMS_LED -> Net-(R24-Pad2)
Routing:
- net /connector/SHOULDER_OUT: track 255.8 -> 0.00 mm, vias 5 -> 0
- net /connector/DRIVER_OUTPUT_LED: track 0.00 -> 165.2 mm, vias 0 -> 6
- net /connector/SHOULDER_OUT_LED: track 0.00 -> 160.2 mm, vias 0 -> 3
- net Net-(U5A-Q): track 0.00 -> 111.8 mm, vias 0 -> 6
- net /3.3V: track 543.1 -> 593.2 mm, vias 17 -> 21
- net /connector/ECU_OK: track 130.2 -> 175.4 mm
- net /connector/AIR_POWER: track 142.0 -> 187.1 mm, vias 4 -> 3
- net /3.3V_PDOC: track 178.7 -> 223.1 mm, vias 6 -> 10
- net /connector/MC_OK_INDICATOR: track 137.3 -> 93.9 mm
- net /AIR_OUTPUT/DRIVER_OUTPUT: track 225.8 -> 184.9 mm
- net /connector/CRASH_SENSOR_MONITOR: track 169.8 -> 208.5 mm
- net GND: track 143.0 -> 178.8 mm, vias 74 -> 97
- net /connector/LEFT_ESTOP_OUT: track 144.2 -> 177.1 mm
- net Net-(R47-Pad2): track 0.00 -> 31.4 mm, vias 0 -> 5
- net Net-(R51-Pad2): track 0.00 -> 31.2 mm, vias 0 -> 2
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- added copper zone on F.Cu, net /3.3V
- added copper zone on F.Cu, net /3.3V_0
- added copper zone on F.Cu, net /3.3V_1
- added copper zone on F.Cu, net /3.3V_2
- added copper zone on F.Cu, net /3.3V_PDOC
Other:
- board text removed: "AIR OUT"
