File: shutdownPCB/shutdownPCB.kicad_sch (KiCad schematic)
At the start: 5 parts

Commit message: Updated 12 Sep
Other:
- sheet connector ports: added DRIVER_OUTPUT_LED, SHOULDER_OUT_LED; removed DRIVER_OUTPUT, SHOULDER_OUT
- sheet logic ports: added DRIVER_OUTPUT_LED, SHOULDER_OUT_LED; removed SHOULDER_OUT

Commit message: My last update
Parts:
- renumbered PRES_1 to BREAK_PRESSED1
Changed lines of the file:
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@@
 		(on_board yes)
 		(dnp no)
-		(property "Reference" "PRES_1"
+		(property "Reference" "BREAK_PRESSED1"
 			(at 156.21 217.297 0)
 			(effects
